File: PhasedUltrasonicArray.kicad_pcb (KiCad board)
At the start: 2 copper layers, 84.5 x 25.8 mm, 18 parts, among them J1 Conn_01x12_Pin, J2 Conn_01x02_Socket, U1 TC78H621FNG, U2 TC78H621FNG, U3 TC78H621FNG, U4 TC78H621FNG

Commit message: 1
Parts:
- added G***: LOGO, LOGO, F.Cu at (139.6, 75.7)
